File: esp32s3-rail.kicad_pcb (KiCad board)
At the start: 2 copper layers, 32 x 80 mm, 99 parts, among them J1 Conn_01x06, J2 Conn_01x06, J3 USB_C_Receptacle_USB2.0_16P, J4 RJ45_Wuerth_7499010121A, J5 490107670612, J6 Conn_02x20_Odd_Even, K1 36.11.9.005.4011, K2 36.11.9.005.4011, Q1 AO3400, Q2 AO3400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

Commit message: Update stacking header.
Signed-off-by: Dominik Bayerl <dominik.bayerl@carissma.eu>
Parts:
- removed J1, J2: Conn_01x06, Connector_Phoenix_MSTB:PhoenixContact_MSTBA_2,5_6-G_1x06_P5.00mm_Horizontal
- added J7: Conn_01x12, Connector_Molex:Molex_SPOX_5268-12A_1x12_P2.50mm_Horizontal, F.Cu at (22.5, 93.4)
- moved U4 168.0 mm to (26.7, 48.3), turned to 180 degrees
- moved J3 152.3 mm to (26.7, 24.1), turned to 180 degrees
- moved U5 146.2 mm to (30.5, 63.9)
- moved K2 143.9 mm to (22.1, 75.5)
- moved U2 132.7 mm to (47.0, 54.6)
- moved U1 105.0 mm to (44.8, 62.3), turned to -90 degrees
- moved K1 104.8 mm to (37.8, 75.5)
- moved J4 69.3 mm to (37.1, 40.1), turned to 90 degrees
- moved J6 54.0 mm to (78.7, 30.5)
Routing:
- net /relay1/11: track 0.00 -> 23.5 mm
- net /relay/11: track 0.00 -> 20.6 mm
- net /relay/14: track 0.00 -> 10.4 mm
- net /relay1/14: track 0.00 -> 7.81 mm
